Commit message: Update lfb.xacro

File: line_follower/urdf/lfb.xacro (robot description, xacro)
@@ -14,5 +14,5 @@
       <origin xyz="-0.032 0 0.0" rpy="0 0 0"/>
       <geometry>
-        <mesh filename="$(find line_follower)/urdf/meshes/burger_base.stl" scale="0.001 0.001 0.001"/>
+        <mesh filename="$(find line_follower)/urdf/meshes/lfb_base.stl" scale="0.001 0.001 0.001"/>
       </geometry>
       <material name="light_black"/>
